File: KiCad/power.kicad_sch (KiCad schematic)
At the start: 5 parts, among them K1 SRD-05VDC-SL-C, Q5 NMOS

Commit message: delete pwm, add 12 neopixel outputs
Other:
- note added: "min. 500mA power consumption"
Changed lines of the file:
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@@
 	(generator_version "10.0")
 	(paper "A4")
+	(text "min. 500mA power consumption"
+		(exclude_from_sim no)
+		(at 99.0357 73.5817 0)
+		(effects
+			(font
+				(size 1.27 1.27)
+			)
+		)
+	)
 	(junction
 		(at 87.63 52.07)

Commit message: work on new design
Parts:
- added F1: Fuse, Fuse:Fuseholder_Blade_Mini_Keystone_3568, symbol Device:Fuse
- Q5: value NMOS -> AO3400A; footprint (none) -> Package_TO_SOT_SMD:SOT-23; LCSC (none) -> C20917
- R22: LCSC (none) -> C2907294
Connections:
- net +24V: now also F1.1; no longer K1.1
- new net: F1.2, K1.1
Other:
- moved on the sheet: D2, K1, Q5, R21, R22
