File: KiCad/LEDController.kicad_sch (KiCad schematic)
At the start: 42 parts, among them SW1 BOOT, SW2 EN, U1 TPS54202DDC, U2 ESP32-S3-WROOM-2, U3 TPS54202DDC

Commit message: arrange components
Other:
- moved on the sheet: C10, C11, C6, C7, C8, C9, L1, R10, R11, R12, U1
