File: KiCad/outputs.kicad_sch (KiCad schematic)
At the start: 39 parts, among them J1 UART, J10 LED2, J13 LED3, J14 LED4, J15 LED8, J16 LED7, J17 LED6, J18 LED5, J19 LED9, J20 LED10, J21 LED11, J22 LED12, J4 Conn_01x02, J5 Conn_01x02, J6 USB_C_Receptacle_USB2.0_16P, J7 Conn_01x14, J8 JTAG, J9 LED1, U7 SN74LVC8T245, U8 SN74LVC8T245

Commit message: arrange components
Parts:
- J10, J13, J14, J15, J16, J17, J18, J19, J20, J21, J22, J9: footprint TerminalBlock_Phoenix:TerminalBlock_Phoenix_MKDS-3-3-5.08_1x03_P5.08mm_Horizontal -> CONN-TH_3P-P5.08_WJ2EDGRC-5.08-3P; LCSC (none) -> C8377
- J4: value Conn_01x02 -> 5V; footprint TerminalBlock_Phoenix:TerminalBlock_Phoenix_MKDS-3-2-5.08_1x02_P5.08mm_Horizontal -> Library:CONN-TH_HB9500M-9.5-2P; LCSC (none) -> C601239
- J5: value Conn_01x02 -> 24V; footprint TerminalBlock_Phoenix:TerminalBlock_Phoenix_MKDS-3-2-5.08_1x02_P5.08mm_Horizontal -> Library:CONN-TH_HB9500M-9.5-2P; LCSC (none) -> C601239
Connections:
- net +24V: no longer D3.1 (K), J4.1 (Pin_1)
- net +5V: now also D3.1 (K), J4.1 (Pin_1)
